File: schematic/blink1mk3_micro1a.sch (EAGLE design)
At the start: 36 parts, among them J1 NONPOP, U1 EFM32HG309F64G, X1 USBPCB2, X2 USBPCB2, X3 USBPCB2

Commit message: sync schematic experiments
Parts:
- removed C10, C11, C5, C6, C7, C8, C9: 0.1uF, adafruit:C-USC0603
- removed GND: TPTP14SQ, testpad:TPTP14SQ
- removed J1: NONPOP, SparkFun-Connectors:USB_MICRO-B_FEMALE-SMT
- removed LED3, LED4, LED5, LED6, LED7, LED8, LED9: SK6812MINI, adafruit:WS2812B3535
- removed LERX, LETX: TPTP15R, testpad:TPTP15R
- removed U$1: LED_STRIP_3P, NeoJoints:LED_STRIP_3P
- removed X1, X3: USBPCB2, todstuff:USBPCB2
- 5V, C, D: value TPTP15R -> TPTP10R; device testpad:TPTP15R -> testpad:TPTP10R
- C1, C2, C3, C4: device adafruit:C-USC0603 -> adafruit:C-USC0402
- G: value TPTP14SQ -> TPTP10R; device testpad:TPTP14SQ -> testpad:TPTP10R
- LED1, LED2: value SK6812MINI -> WS2812B4020SIDE; device adafruit:WS2812B3535 -> todstuff:WS2812B4020SIDE
- R3, R4: device adafruit:R-US_R0603 -> adafruit:R-US_R0402
Connections:
- removed net N$10: LED6.DO, LED7.DI
- removed net N$4: LED7.DO, LED8.DI
- removed net N$5: LED4.DO, LED5.DI
- removed net N$6: LED5.DO, LED6.DI
- removed net N$7: LED2.DO, LED3.DI
- removed net N$8: LED3.DO, LED4.DI
- removed net N$9: LED8.DO, LED9.DI
- net +5V: no longer C10.1, C11.1, C5.1, C6.1, C7.1, C8.1, C9.1, J1.VBUS, LED3.VDD, LED4.VDD, LED5.VDD, LED6.VDD, LED7.VDD, LED8.VDD, LED9.VDD, U$1.A
- net DO: now also LED2.DO; no longer LED9.DO, U$1.B
- net GND: no longer C10.2, C11.2, C5.2, C6.2, C7.2, C8.2, C9.2, GND.TP, J1.GND, LED3.GND, LED4.GND, LED5.GND, LED6.GND, LED7.GND, LED8.GND, LED9.GND, U$1.C
- net LEUO_RX: no longer LERX.TP
- net LEUO_TX: no longer LETX.TP
- net USB_D+: no longer J1.D+
- net USB_D-: no longer J1.D-
Other:
- moved on the sheet: 5V, C4, D1, G, X2
