File: schematic/blink1mk3_card1.sch (EAGLE design)
At the start: 15 parts, among them U1 EFM32HG309F64G, X2 USBPCB2

Commit message: added business card idea
Parts:
- added C10, C11, C5, C6, C7, C8, C9: 0.1uF, adafruit:C-USC0603
- added GND: TPTP14SQ, testpad:TPTP14SQ
- added J1: NONPOP, SparkFun-Connectors:USB_MICRO-B_FEMALE-SMT
- added LED3, LED4, LED5, LED6, LED7, LED8, LED9: SK6812MINI, adafruit:WS2812B3535
- added PA0, PB11, PB8, RX, TX: TPTP15R, testpad:TPTP15R
- added U$1: LED_STRIP_3P, NeoJoints:LED_STRIP_3P
- added X1, X3: USBPCB2, todstuff:USBPCB2
- 5V, C, D: value TPTP10R -> TPTP15R; device testpad:TPTP10R -> testpad:TPTP15R
- C1, C2, C3, C4: device adafruit:C-USC0402 -> adafruit:C-USC0603
- G: value TPTP10SQ -> TPTP14SQ; device testpad:TPTP10SQ -> testpad:TPTP14SQ
- LED1, LED2: value WS2812B4020SIDE -> SK6812MINI; device todstuff:WS2812B4020SIDE -> adafruit:WS2812B3535
- R3, R4: device adafruit:R-US_R0402 -> adafruit:R-US_R0603
Connections:
- removed net LED1: U1.PA0
- removed net N$1: U1.PB11
- removed net N$3: U1.PB8
- new net N$10: LED6.DO, LED7.DI
- new net N$4: LED7.DO, LED8.DI
- new net N$5: LED4.DO, LED5.DI
- new net N$6: LED5.DO, LED6.DI
- new net N$7: LED2.DO, LED3.DI
- new net N$8: LED3.DO, LED4.DI
- new net N$9: LED8.DO, LED9.DI
- new net PA0: PA0.TP, U1.PA0
- new net PB11: PB11.TP, U1.PB11
- new net PB8: PB8.TP, U1.PB8
- net +5V: now also C10.1, C11.1, C5.1, C6.1, C7.1, C8.1, C9.1, J1.VBUS, LED3.VDD, LED4.VDD, LED5.VDD, LED6.VDD, LED7.VDD, LED8.VDD, LED9.VDD, U$1.A
- net DO: now also LED9.DO, U$1.B; no longer LED2.DO
- net GND: now also C10.2, C11.2, C5.2, C6.2, C7.2, C8.2, C9.2, GND.TP, J1.GND, LED3.GND, LED4.GND, LED5.GND, LED6.GND, LED7.GND, LED8.GND, LED9.GND, U$1.C
- net LEUO_RX: now also RX.TP
- net LEUO_TX: now also TX.TP
- net USB_D+: now also J1.D+
- net USB_D-: now also J1.D-
Other:
- moved on the sheet: 5V, C4, D1, G, X2
