File: schematic/blink1mk3_micro1c.sch (EAGLE design)
At the start: 15 parts, among them U1 EFM32HG309F64G, X1 USBPCB2

Commit message: fix EFM32HG309 pad spacing issue. omg what a slog
Parts:
- added TOUCH: TPTP10R, testpad:TPTP10R
- D1: value (none) -> 1N4148
Connections:
- net CAP0A: now also TOUCH.TP
Other:
- moved on the sheet: C4, D1
