File: schematic/blink1mk3_005t6_4L.brd (EAGLE design)
At the start: 15.5 x 13.7 mm, 19 parts, among them T0A TPTP15R, T1B TPTP15R, U1 EFM32HG309F64G, X1 USB

Commit message: rename sch 005t6_5050_4l to 005t6_4L
Parts:
- LED1, LED2: value SK6812MINI -> SK6812
Changed lines of the file:
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@@
 <?xml version="1.0" encoding="utf-8"?>
 <!DOCTYPE eagle SYSTEM "eagle.dtd">
-<eagle version="9.4.2">
+<eagle version="9.5.0">
 <drawing>
 <settings>
@@
 <attribute name="VALUE" x="11.049" y="-5.842" size="1.27" layer="28" rot="MR0"/>
 </element>
-<element name="LED1" library="adafruit" library_urn="urn:adsk.eagle:library:420" package="WS2812B" value="SK6812MINI" x="9.556" y="0" smashed="yes" rot="R270">
+<element name="LED1" library="adafruit" library_urn="urn:adsk.eagle:library:420" package="WS2812B" value="SK6812" x="9.556" y="0" smashed="yes" rot="R270">
 <attribute name="NAME" x="10.964" y="0.408" size="0.8" layer="25" ratio="12" rot="R180"/>
 <attribute name="VALUE" x="7.016" y="1.778" size="0.4064" layer="27" ratio="10" rot="R270"/>
 </element>
-<element name="LED2" library="adafruit" library_urn="urn:adsk.eagle:library:420" package="WS2812B" value="SK6812MINI" x="9.544" y="0" smashed="yes" rot="MR270">
+<element name="LED2" library="adafruit" library_urn="urn:adsk.eagle:library:420" package="WS2812B" value="SK6812" x="9.544" y="0" smashed="yes" rot="MR270">
 <attribute name="NAME" x="10.833" y="-0.335" size="0.8" layer="26" ratio="12" rot="MR0"/>
 <attribute name="VALUE" x="12.084" y="1.778" size="0.4064" layer="28" ratio="10" rot="MR270"/>
