File: schematic/blink1mk3_005t6_4L.sch (EAGLE design)
At the start: 19 parts, among them T0A TPTP15R, T1B TPTP15R, U1 EFM32HG309F64G, X1 USB

Commit message: rename sch 005t6_5050_4l to 005t6_4L
Parts:
- LED1, LED2: value SK6812MINI -> SK6812
Changed lines of the file:
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@@
 <?xml version="1.0" encoding="utf-8"?>
 <!DOCTYPE eagle SYSTEM "eagle.dtd">
-<eagle version="9.4.2">
+<eagle version="9.5.0">
 <drawing>
 <settings>
@@
 <part name="P+3" library="supply1" deviceset="+5V" device=""/>
 <part name="GND1" library="SparkFun-20110517" deviceset="GND" device=""/>
-<part name="LED1" library="adafruit" library_urn="urn:adsk.eagle:library:420" deviceset="WS2812B" device="5050" value="SK6812MINI"/>
-<part name="LED2" library="adafruit" library_urn="urn:adsk.eagle:library:420" deviceset="WS2812B" device="5050" value="SK6812MINI"/>
+<part name="LED1" library="adafruit" library_urn="urn:adsk.eagle:library:420" deviceset="WS2812B" device="5050" value="SK6812"/>
+<part name="LED2" library="adafruit" library_urn="urn:adsk.eagle:library:420" deviceset="WS2812B" device="5050" value="SK6812"/>
 <part name="G" library="testpad" library_urn="urn:adsk.eagle:library:385" deviceset="TP" device="TP10R" package3d_urn="urn:adsk.eagle:package:27959/1" value="TPTP10R"/>
 <part name="+5" library="testpad" library_urn="urn:adsk.eagle:library:385" deviceset="TP" device="TP10R" package3d_urn="urn:adsk.eagle:package:27959/1" value="TPTP10R"/>
