File: schematic/blink1mk3_005t6_5050_4l_usbc.brd (EAGLE design)
At the start: 18.9 x 10.4 mm, 19 parts, among them J1 DX07P024AJ1R1500, T0A TPTP15R, T1B TPTP15R, U1 EFM32HG309F64G

Commit message: rename sch 005t6_5050_4l to 005t6_4L
Parts:
- R1, R2: device adafruit:R0402 -> rcl:R0402
- moved R1 0.10 mm to (0.30, 0.50)
Other:
- outline, holes or cut-outs redrawn
Changed lines of the file:
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@@
 <?xml version="1.0" encoding="utf-8"?>
 <!DOCTYPE eagle SYSTEM "eagle.dtd">
-<eagle version="9.4.2">
+<eagle version="9.5.0">
 <drawing>
 <settings>
@@
 </layers>
 <board>
-<fusionsync huburn="a.cGVyc29uYWw6dWUyOWMzMmM3" projecturn="a.cGVyc29uYWw6dWUyOWMzMmM3IzIwMTgwNDI3MTI5NTI4MDU2" f3durn="urn:adsk.wipprod:dm.lineage:oQMhUYtWTpi6h9pgRYsZEQ" pcbguid="654822f9-e281-4680-880e-41f5a54f4fc1" lastpulledtime="" lastsyncedchangeguid="63d708ea-91a7-6766-def3-66ee2e413c6e"/>
+<fusionsync huburn="a.cGVyc29uYWw6dWUyOWMzMmM3" projecturn="a.cGVyc29uYWw6dWUyOWMzMmM3IzIwMTgwNDI3MTI5NTI4MDU2" f3durn="urn:adsk.wipprod:dm.lineage:oQMhUYtWTpi6h9pgRYsZEQ" pcbguid="654822f9-e281-4680-880e-41f5a54f4fc1" lastpulledtime="" lastsyncedchangeguid="ad1f8c0a-0a65-18ea-7cef-00f3a15e6fd9"/>
 <plain>
 <text x="4.4164625" y="-3.1435625" size="0.8" layer="21" ratio="12" rot="SR90">thingm.com</text>
@@
 <dimension x1="-7.1" y1="-3.9" x2="-1.9" y2="4.3" x3="-12.867190625" y3="0.2" textsize="0.3048" layer="47" dtype="vertical" width="0.0254" visible="yes"/>
 <dimension x1="-6.2" y1="-3.9" x2="-4.4" y2="3.9" x3="-11.867190625" y3="0" textsize="0.3048" layer="47" dtype="vertical" width="0.0254" visible="yes"/>
-<wire x1="-1.6" y1="4.3" x2="0.2" y2="4.3" width="0.127" layer="20"/>
+<wire x1="-1.5" y1="4.3" x2="0.2" y2="4.3" width="0.127" layer="20"/>
 <wire x1="0.2" y1="4.3" x2="0.2" y2="4.565" width="0.127" layer="20"/>
 <wire x1="0.2" y1="4.565" x2="0.835" y2="5.2" width="0.127" layer="20"/>
@@
 <dimension x1="13.2" y1="-4.2" x2="13.3" y2="-5.2" x3="14.967190625" y3="-4.7" textsize="0.3048" layer="47" dtype="vertical" width="0.0254" visible="yes"/>
 <dimension x1="11.4" y1="5.2" x2="13.9" y2="4.2" x3="14.767190625" y3="4.7" textsize="0.3048" layer="47" dtype="vertical" width="0.0254" visible="yes"/>
-<wire x1="-3.8" y1="3.9" x2="-1.6" y2="3.9" width="0.127" layer="20"/>
+<wire x1="-3.8" y1="3.9" x2="-1.5" y2="3.9" width="0.127" layer="20"/>
 <wire x1="-4.15" y1="3.56" x2="-3.8" y2="3.9" width="0.127" layer="20"/>
 <wire x1="-4.3" y1="3" x2="-4.15" y2="3.08" width="0.127" layer="20" curve="90"/>
@@
 <wire x1="-4.6" y1="3" x2="-4.3" y2="3" width="0.127" layer="20"/>
 <wire x1="-4.15" y1="3.08" x2="-4.15" y2="3.56" width="0.127" layer="20"/>
-<wire x1="-1.6" y1="4.3" x2="-1.6" y2="3.9" width="0.127" layer="20"/>
+<wire x1="-1.5" y1="4.3" x2="-1.5" y2="3.9" width="0.127" layer="20"/>
+<dimension x1="-4.8" y1="4.2" x2="-1.5" y2="4.644" x3="-3.15" y3="8.999" textsize="0.254" layer="47" dtype="horizontal" width="0.0254" visible="yes"/>
 </plain>
 <attributes>
@@
 <attribute name="VALUE" x="-0.335" y="-0.205" size="1.27" layer="27"/>
 </element>
-<element name="R1" library="adafruit" library_urn="urn:adsk.eagle:library:420" package="R0402" package3d_urn="urn:adsk.eagle:package:6240564/1" value="15" x="0.3" y="0.6" smashed="yes" rot="R180">
-<attribute name="NAME" x="1.471" y="0.225" size="0.8" layer="25" ratio="12"/>
-<attribute name="VALUE" x="0.935" y="2.632" size="1.27" layer="27" rot="R180"/>
-</element>
-<element name="R2" library="adafruit" library_urn="urn:adsk.eagle:library:420" package="R0402" package3d_urn="urn:adsk.eagle:package:6240564/1" value="15" x="0.3" y="-0.6" smashed="yes" rot="R180">
-<attribute name="NAME" x="1.471" y="-0.96" size="0.8" layer="25" ratio="12"/>
-<attribute name="VALUE" x="0.935" y="1.432" size="1.27" layer="27" rot="R180"/>
-</element>
 <element name="D" library="testpad" library_urn="urn:adsk.eagle:library:385" package="TP10R" package3d_urn="urn:adsk.eagle:package:27959/1" value="TPTP10R" x="10.7" y="4" smashed="yes" rot="MR0">
 <attribute name="NAME" x="9.792" y="3.646" size="0.8" layer="26" ratio="12" rot="MR0"/>
@@
 <attribute name="NAME" x="1.411" y="-2.167" size="0.8128" layer="25" ratio="12"/>
 <attribute name="VALUE" x="0.935" y="0.232" size="1.27" layer="27" rot="R180"/>
+</element>
+<element name="R1" library="rcl" library_urn="urn:adsk.eagle:library:334" package="R0402" package3d_urn="urn:adsk.eagle:package:23547/3" value="15" x="0.3" y="0.5" smashed="yes" rot="R180">
+<attribute name="NAME" x="0.935" y="-0.135" size="1.27" layer="25" rot="R180"/>
+<attribute name="POPULARITY" value="34" x="0.3" y="0.5" size="1.778" layer="27" rot="R180" display="off"/>
+<attribute name="SPICEPREFIX" value="R" x="0.3" y="0.5" size="1.778" layer="27" rot="R180" display="off"/>
+<attribute name="VALUE" x="0.935" y="2.405" size="1.27" layer="27" rot="R180"/>
+</element>
+<element name="R2" library="rcl" library_urn="urn:adsk.eagle:library:334" package="R0402" package3d_urn="urn:adsk.eagle:package:23547/3" value="15" x="0.3" y="-0.6" smashed="yes" rot="R180">
+<attribute name="NAME" x="0.935" y="-1.235" size="1.27" layer="25" rot="R180"/>
+<attribute name="POPULARITY" value="34" x="0.3" y="-0.6" size="1.778" layer="27" rot="R180" display="off"/>
+<attribute name="SPICEPREFIX" value="R" x="0.3" y="-0.6" size="1.778" layer="27" rot="R180" display="off"/>
+<attribute name="VALUE" x="0.935" y="1.305" size="1.27" layer="27" rot="R180"/>
 </element>
 </elements>
@@
 <signal name="RUSB_D+">
 <contactref element="U1" pad="18"/>
-<contactref element="R2" pad="1"/>
 <via x="6.3792" y="2.702" extent="1-16" drill="0.35"/>
 <wire x1="5.865425" y1="3.215775" x2="6.3792" y2="2.702" width="0.2032" layer="16"/>
@@
 <wire x1="5.515775" y1="3.215775" x2="5.865425" y2="3.215775" width="0.2032" layer="16"/>
 <wire x1="5.308" y1="3.008" x2="5.515775" y2="3.215775" width="0.2032" layer="16"/>
-<wire x1="6.3792" y1="2.702" x2="3.0772" y2="-0.6" width="0.2032" layer="1"/>
-<wire x1="3.0772" y1="-0.6" x2="0.95" y2="-0.6" width="0.2032" layer="1"/>
+<wire x1="3.0772" y1="-0.6" x2="6.3792" y2="2.702" width="0.2032" layer="1"/>
+<contactref element="R2" pad="1"/>
+<wire x1="0.8" y1="-0.6" x2="3.0772" y2="-0.6" width="0.2032" layer="1"/>
 </signal>
 <signal name="RUSB_D-">
 <contactref element="U1" pad="17"/>
-<contactref element="R1" pad="1"/>
 <wire x1="4.658" y1="2.5" x2="4.658" y2="3.21" width="0.2032" layer="16"/>
-<wire x1="0.95" y1="0.6" x2="1.957834375" y2="0.6" width="0.2032" layer="1"/>
 <wire x1="4.658" y1="3.21" x2="4.798" y2="3.35" width="0.2032" layer="16"/>
 <via x="4.798" y="3.35" extent="1-16" drill="0.35"/>
 <wire x1="1.957834375" y1="0.6" x2="4.798" y2="3.35" width="0.2032" layer="1"/>
+<contactref element="R1" pad="1"/>
+<wire x1="0.8" y1="0.5" x2="1.857834375" y2="0.5" width="0.2032" layer="1"/>
+<wire x1="1.857834375" y1="0.5" x2="1.957834375" y2="0.6" width="0.2032" layer="1"/>
 </signal>
 <signal name="USB_D-">
+<contactref element="J1" pad="A7"/>
 <contactref element="R1" pad="2"/>
-<contactref element="J1" pad="A7"/>
-<wire x1="-1.45" y1="0.25" x2="-1.1" y2="0.6" width="0.1524" layer="1"/>
-<wire x1="-1.1" y1="0.6" x2="-0.35" y2="0.6" width="0.1524" layer="1"/>
-<wire x1="-2.925" y1="0.25" x2="-1.45" y2="0.25" width="0.1524" layer="1"/>
+<wire x1="-2.925" y1="0.25" x2="-1.25" y2="0.25" width="0.1524" layer="1"/>
+<wire x1="-1.25" y1="0.25" x2="-1.05" y2="0.25" width="0.2032" layer="1"/>
+<wire x1="-1.05" y1="0.25" x2="-0.8" y2="0.5" width="0.2032" layer="1"/>
+<wire x1="-0.8" y1="0.5" x2="-0.2" y2="0.5" width="0.2032" layer="1"/>
 </signal>
 <signal name="USB_D+">
-<contactref element="R2" pad="2"/>
 <contactref element="J1" pad="A6"/>
 <wire x1="-1.45" y1="-0.25" x2="-1.1" y2="-0.6" width="0.1524" layer="1"/>
-<wire x1="-1.1" y1="-0.6" x2="-0.35" y2="-0.6" width="0.1524" layer="1"/>
 <wire x1="-2.925" y1="-0.25" x2="-1.45" y2="-0.25" width="0.1524" layer="1"/>
+<contactref element="R2" pad="2"/>
+<wire x1="-1.1" y1="-0.6" x2="-0.2" y2="-0.6" width="0.2032" layer="1"/>
 </signal>
 <signal name="DECOUPLE">
