File: schematic/blink1mk3_005t6_5050_4l_usbc.sch (EAGLE design)
At the start: 19 parts, among them J1 DX07P024AJ1R1500, T0A TPTP15R, T1B TPTP15R, U1 EFM32HG309F64G

Commit message: rename sch 005t6_5050_4l to 005t6_4L
Parts:
- R1, R2: device adafruit:R-US_R0402 -> rcl:R-US_R0402
